File: dc_power.kicad_sch (KiCad schematic)
At the start: 42 parts, among them J2 DCJ200-10-A-XX-K_REVA, U1 NCP1117-3.3_SOT223, U11 TC7662BCOA713, U2 TPS54302, U3 LDFMPUR, U9 TPS54302

Commit message: added some badass comments
Other:
- note added: "DACs, LEDs, VOltage/Current Sense, OLED"
- note added: "Nano supply"
- note added: "OP amp supply"
- note added: "Transformer output"
